File: board/lab.brd (EAGLE design)
At the start: 53 x 66 mm, 7 parts

Commit message: add user_button
Parts:
- added S3: (no value), switch-omron:B3F-10XX
Connections:
- new net IO16: S3.1, S3.2, U$1.P$27
- net GND: now also S3.3, S3.4
Routing:
- net IO16: track 0.00 -> 12.6 mm
Changed lines of the file:
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@@
 <element name="R4" library="rcl" package="0207/10" value="10k" x="3.81" y="33.02" rot="R90"/>
 <element name="U$1" library="esp32-devkit" package="ESP32_DEVKITC" value="ESP32_DEVKITC" x="26.67" y="30.48"/>
+<element name="S3" library="switch-omron" package="B3F-10XX" value="" x="46.99" y="24.13" rot="R90">
+<attribute name="MPN" value="B3F-1000" x="46.99" y="24.13" size="1.778" layer="27" rot="R90" display="off"/>
+<attribute name="MF" value="" x="46.99" y="24.13" size="1.778" layer="27" rot="R90" display="off"/>
+<attribute name="OC_NEWARK" value="36M3542" x="46.99" y="24.13" size="1.778" layer="27" rot="R90" display="off"/>
+<attribute name="OC_FARNELL" value="176432" x="46.99" y="24.13" size="1.778" layer="27" rot="R90" display="off"/>
+</element>
 </elements>
 <signals>
@@
 <vertex x="-6.35" y="71.12"/>
 </polygon>
+<contactref element="S3" pad="3"/>
+<contactref element="S3" pad="4"/>
 </signal>
 <signal name="+3V3">
@@
 <via x="5" y="61" extent="1-16" drill="3" diameter="6"/>
 </signal>
+<signal name="IO16">
+<contactref element="S3" pad="1"/>
+<contactref element="S3" pad="2"/>
+<contactref element="U$1" pad="P$27"/>
+<wire x1="39.37" y1="26.67" x2="44.7294" y2="26.67" width="0.4064" layer="1"/>
+<wire x1="44.7294" y1="26.67" x2="44.7294" y2="27.3812" width="0.4064" layer="1"/>
+<wire x1="44.7294" y1="27.3812" x2="44.7294" y2="20.8788" width="0.4064" layer="1"/>
+</signal>
 </signals>

Commit message: change ADCpin A18 -> A4
Connections:
- removed net A18: JP2.2, R4.2, U$1.P$11
- new net A4: JP2.2, R4.2, U$1.P$13
Routing:
- net A18: track 16.8 -> 0.00 mm
- net A4: track 0.00 -> 15.8 mm
Changed lines of the file:
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@@
 <wire x1="12.7" y1="31.75" x2="13.97" y2="31.75" width="0.4064" layer="1"/>
-</signal>
-<signal name="A18">
-<contactref element="U$1" pad="P$11"/>
-<contactref element="JP2" pad="2"/>
-<contactref element="R4" pad="2"/>
-<wire x1="3.81" y1="38.1" x2="3.81" y2="43.18" width="0.4064" layer="1"/>
-<wire x1="13.97" y1="34.29" x2="7.62" y2="34.29" width="0.4064" layer="1"/>
-<wire x1="7.62" y1="34.29" x2="3.81" y2="38.1" width="0.4064" layer="1"/>
 </signal>
 <signal name="A5">
@@
 <wire x1="44.7294" y1="27.3812" x2="44.7294" y2="20.8788" width="0.4064" layer="1"/>
 </signal>
+<signal name="A4">
+<contactref element="U$1" pad="P$13"/>
+<contactref element="JP2" pad="2"/>
+<contactref element="R4" pad="2"/>
+<wire x1="3.81" y1="38.1" x2="3.81" y2="43.18" width="0.4064" layer="1"/>
+<wire x1="3.81" y1="38.1" x2="5.08" y2="39.37" width="0.4064" layer="16"/>
+<wire x1="5.08" y1="39.37" x2="13.97" y2="39.37" width="0.4064" layer="16"/>
+</signal>
 </signals>
